File: armpcb.kicad_sch (KiCad schematic)
At the start: 0 parts

Commit message: changing naming conventions
Parts:
- added F1, F2, F3, F4, F5, F6, F7: Fuse, Fuse:Fuse_Blade_ATO_directSolder, symbol Device:Fuse
- added H1, H2, H3, H4: MountingHole_Pad, MountingHole:MountingHole_2.2mm_M2_Pad, symbol Mechanical:MountingHole_Pad
- added J1, J4: Screw_Terminal_01x02, TerminalBlock_Phoenix:TerminalBlock_Phoenix_MKDS-1,5-2_1x02_P5.00mm_Horizontal, symbol Connector:Screw_Terminal_01x02
- added J2: Screw_Terminal_01x06, TerminalBlock_Phoenix:TerminalBlock_Phoenix_MKDS-1,5-6_1x06_P5.00mm_Horizontal, symbol Connector:Screw_Terminal_01x06
- added J3: Screw_Terminal_01x08, TerminalBlock_Phoenix:TerminalBlock_Phoenix_MKDS-1,5-8_1x08_P5.00mm_Horizontal, symbol Connector:Screw_Terminal_01x08
- added J5, J6: Conn_01x02_Socket, Connector_PinSocket_2.54mm:PinSocket_1x02_P2.54mm_Vertical, symbol Connector:Conn_01x02_Socket
- added J7: USB_C_Receptacle_USB2.0_14P, Connector_USB:USB_C_Receptacle_GCT_USB4105-xx-A_16P_TopMnt_Horizontal, symbol Connector:USB_C_Receptacle_USB2.0_14P
- added P1: USB_C_Plug_USB2.0, Connector_USB:USB_C_Plug_ShenzhenJingTuoJin_918-118A2021Y40002_Vertical, symbol Connector:USB_C_Plug_USB2.0
Connections:
- new net: F4.1, J3.2 (Pin_2)
- new net: F3.1, J3.4 (Pin_4)
- new net: F2.1, J3.6 (Pin_6)
- new net: F1.1, J3.8 (Pin_8)
- new net: J7.A1 (GND), J7.A12 (GND), J7.B1 (GND), J7.B12 (GND), P1.A1 (GND), P1.A12 (GND), P1.B1 (GND), P1.B12 (GND)
- new net: J7.A4 (VBUS), J7.A9 (VBUS), J7.B4 (VBUS), J7.B9 (VBUS), P1.A4 (VBUS), P1.A9 (VBUS), P1.B4 (VBUS), P1.B9 (VBUS)
- new net: J7.A5 (CC1), P1.A5 (CC)
- new net: J7.A6 (D+), J7.B6 (D+), P1.A6 (D+)
- new net: J7.A7 (D-), J7.B7 (D-), P1.A7 (D-)
- new net: J7.B5 (CC2), P1.B5 (VCONN)
- new net: J7.SH (SHIELD), P1.SH (SHIELD)
- new net: J5.2 (Pin_2), J6.1 (Pin_1)
- new net: J5.1 (Pin_1), J6.2 (Pin_2)
- new net: F5.2, J2.1 (Pin_1)
- new net: F6.2, J2.3 (Pin_3)
- new net: F7.2, J2.5 (Pin_5)
- new net +12V0: F5.1, F6.1, F7.1, J4.1 (Pin_1)
- new net +24V0: F1.2, F2.2, F3.2, F4.2, J1.1 (Pin_1)
- new net GND1: H1.1, H4.1, J1.2 (Pin_2), J3.1 (Pin_1), J3.3 (Pin_3), J3.5 (Pin_5), J3.7 (Pin_7)
- new net GND2: H2.1, H3.1, J2.2 (Pin_2), J2.4 (Pin_4), J2.6 (Pin_6), J4.2 (Pin_2)
